File: MadrinTrack2.sch (KiCad schematic (older format))
At the start: 24 parts, among them J1 Jumper_NC_Small, J2 Conn_01x02_Male, P1 Conn_01x02_Male, P2 Conn_01x02_Male, P4 Conn_01x07_Male, Q1 2N7000, SW1 SW_Push, SW2 SW_Push, U1 DWM1001, U2 MCP73831-2-OT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

Commit message: adding fiducial
Parts:
- added FID1, FID2, FID3: Fiducial, Fiducial:Fiducial_0.75mm_Mask1.5mm, symbol Mechanical:Fiducial
Changed lines of the file:
@@
 Wire Wire Line
 	5800 3750 5975 3750
+$Comp
+L Mechanical:Fiducial FID1
+U 1 1 60601C51
+P 10200 5475
+F 0 "FID1" H 10285 5521 50  0000 L CNN
+F 1 "Fiducial" H 10285 5430 50  0000 L CNN
+F 2 "Fiducial:Fiducial_0.75mm_Mask1.5mm" H 10200 5475 50  0001 C CNN
+F 3 "~" H 10200 5475 50  0001 C CNN
+	1    10200 5475
+	1    0    0    -1
+$EndComp
+$Comp
+L Mechanical:Fiducial FID2
+U 1 1 60602567
+P 10200 5675
+F 0 "FID2" H 10285 5721 50  0000 L CNN
+F 1 "Fiducial" H 10285 5630 50  0000 L CNN
+F 2 "Fiducial:Fiducial_0.75mm_Mask1.5mm" H 10200 5675 50  0001 C CNN
+F 3 "~" H 10200 5675 50  0001 C CNN
+	1    10200 5675
+	1    0    0    -1
+$EndComp
+$Comp
+L Mechanical:Fiducial FID3
+U 1 1 6060289C
+P 10200 5875
+F 0 "FID3" H 10285 5921 50  0000 L CNN
+F 1 "Fiducial" H 10285 5830 50  0000 L CNN
+F 2 "Fiducial:Fiducial_0.75mm_Mask1.5mm" H 10200 5875 50  0001 C CNN
+F 3 "~" H 10200 5875 50  0001 C CNN
+	1    10200 5875
+	1    0    0    -1
+$EndComp
 $EndSCHEMATC
